File: RoadrunnerVmaxModule01.kicad_pcb (KiCad board)
At the start: 2 copper layers, 120 x 90 mm, 3 parts, among them M1 Module-power_12and5V-0.3, M2 Module-mega-mcu144-0.7, M3 Module-input-0.1

Commit message: 5
Parts:
- removed M2: Module-mega-mcu144-0.7, 0.7:mega-mcu144
- removed M3: Module-input-0.1, 0.1:input
- M1: value Module-power_12and5V-0.3 -> Module-mega-mcu144-0.7; footprint 0.3:power_12and5V -> 0.7:mega-mcu144
- moved M1 31.6 mm to (144.2, 103.1)
Connections:
- M1 pad S1: Net-(M1-GND) -> unconnected-(M1-IN_D4-PadS1)
