File: RoadrunnerVmaxModule01.kicad_sch (KiCad schematic)
At the start: 3 parts, among them M1 Module-power_12and5V-0.3, M2 Module-mega-mcu144-0.7, M3 Module-input-0.1

Commit message: Rev a initial board layout
Parts:
- M1: footprint hellen-one-power_12and5V-0.3:power_12and5V -> 0.3:power_12and5V
Changed lines of the file:
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@@
 	(wire
 		(pts
-			(xy 63.5 82.55) (xy 63.5 73.66)
+			(xy 63.5 73.66) (xy 63.5 81.28)
 		)
 		(stroke
@@
 	(wire
 		(pts
-			(xy 26.67 86.36) (xy 26.67 82.55)
+			(xy 78.74 264.16) (xy 78.74 81.28)
 		)
 		(stroke
@@
 	(wire
 		(pts
-			(xy 78.74 264.16) (xy 78.74 86.36)
+			(xy 105.41 264.16) (xy 78.74 264.16)
 		)
 		(stroke
@@
 	(wire
 		(pts
-			(xy 105.41 264.16) (xy 78.74 264.16)
-		)
-		(stroke
-			(width 0)
-			(type default)
-		)
-	)
-	(wire
-		(pts
-			(xy 26.67 82.55) (xy 63.5 82.55)
-		)
-		(stroke
-			(width 0)
-			(type default)
-		)
-	)
-	(wire
-		(pts
-			(xy 78.74 86.36) (xy 26.67 86.36)
+			(xy 78.74 81.28) (xy 63.5 81.28)
 		)
 		(stroke
@@
 			)
 		)
-		(property "Footprint" "hellen-one-power_12and5V-0.3:power_12and5V"
+		(property "Footprint" "0.3:power_12and5V"
 			(at 45.72 41.91 0)
 			(hide yes)

Commit message: 5
Parts:
- removed M1: Module-power_12and5V-0.3, 0.3:power_12and5V, symbol power_12and5V:Module-power_12and5V-0.3
- removed M2: Module-mega-mcu144-0.7, 0.7:mega-mcu144, symbol mega-mcu144:Module-mega-mcu144-0.7
- removed M3: Module-input-0.1, 0.1:input, symbol input:Module-input-0.1
- added M1: Module-mega-mcu144-0.7, 0.7:mega-mcu144, symbol mega-mcu144:Module-mega-mcu144-0.7
