File: RRModule.kicad_pcb (KiCad board)
At the start: 2 copper layers, 120 x 90 mm, 1 part, among them M1 Module-mega-mcu144-0.7

Commit message: 3
Parts:
- added KDFI1: ~, kdFiFootprint:KDFI_V1.4_MODULE, F.Cu at (60.1, 119.9)
- added M2: Module-can-0.1, CAN v0.1:can, F.Cu at (127.3, 67.4)
- added M3: Module-input-0.1, IN v0.1:input, F.Cu at (139.0, 99.5)
- added M4: Module-ign8-0.2, IGN8 v0.2:ign8, F.Cu at (124.0, 88.0)
- added M5: Module-power_12and5V-0.3, PWR v0.3:power_12and5V, F.Cu at (123.0, 123.6)
- moved M1 33.0 mm to (112.5, 70.1), turned to 180 degrees
Connections:
- M1 pad W11: unconnected-(M1-IGN1-PadW11) -> /IGN1
