File: RRModule.kicad_sch (KiCad schematic)
At the start: 1 part, among them M1 Module-mega-mcu144-0.7

Commit message: 3
Parts:
- added KDFI1: ~, kdFiFootprint:KDFI_V1.4_MODULE, symbol k-data Mechanik:KDFI_V1.4_MODULE
- added M2: Module-can-0.1, CAN v0.1:can, symbol can:Module-can-0.1
- added M3: Module-input-0.1, IN v0.1:input, symbol input:Module-input-0.1
- added M4: Module-ign8-0.2, IGN8 v0.2:ign8, symbol ign8:Module-ign8-0.2
- added M5: Module-power_12and5V-0.3, PWR v0.3:power_12and5V, symbol power_12and5V:Module-power_12and5V-0.3
Connections:
- net IGN1: now reaches M1.W11 (IGN1)
- net IGN1: now also M4.V8 (IGN1)
- new net: KDFI1.1-1 (GND@1), KDFI1.5-1 (GND)
- new net: KDFI1.1-7 (+5V), KDFI1.5-2 (+5V)
